File: Sources/Develop/circuit/Alice-F3000/Alice-F3000.sch (KiCad schematic (older format))
At the start: 90 parts, among them J1 XA_4, J2 XA_4, Q1 BSS84, Q10 IPD088N06N3, Q11 IPD088N06N3, Q12 IPD088N06N3, Q2 BSS84, Q3 BSS84, Q4 BSS84, Q9 IPD088N06N3, SW1 SW_DP3T, SW2 SW_Push, SW3 SW_DPDT_x2, U1 74HC595, U12 IR2104, U13 IR2104, U2 74HC595, U3 4_array, U4 4_array, U5 4_array, U6 4_array, U7 OSL10326-LX, U8 OSL10326-LX, U9 ATmega328-AU-MCU_Microchip_AT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, Y1 16MHz

Commit message: 一回目試作機完成
Parts:
- removed SW3: SW_DPDT_x2, symbol Switch:SW_DPDT_x2
- added C19, C21, C26: 100n, Capacitor_SMD:C_0603_1608Metric, symbol Device:C
- added C20: 47u, Capacitor_SMD:C_Elec_6.3x5.4, symbol Device:CP
- added C22, C23, C24, C25: 50V 220uF, Capacitor_SMD:C_Elec_10x10.2, symbol Device:CP
- added C27: 35V 47uF, Capacitor_SMD:C_Elec_10x10.2, symbol Device:CP
- added D11, D12, D13, D14, D15, D19, D20: LED, LED_SMD:LED_0603_1608Metric, symbol Device:LED
- added D18: WS2812B, LED_SMD:LED_WS2812B_PLCC4_5.0x5.0mm_P3.2mm, symbol LED:WS2812B
- added F1: Fuse, Fuse:Fuse_1206_3216Metric, symbol Device:Fuse
- added F2, F3: Fuse, RobotClub_footprint:NR72AB0, symbol Device:Fuse
- added H1, H2, H3, H4: MountingHole_Pad, MountingHole:MountingHole_3mm_Pad_Via, symbol Mechanical:MountingHole_Pad
- added J10, J11, J12, J13, J14, J4, J5, J6, J7, J8, J9: Debug_pin, TestPoint:TestPoint_Loop_D1.80mm_Drill1.0mm_Beaded, symbol Connector:Conn_01x01_Female
- added JP1: Jumper_NC_Dual, Connector_PinHeader_2.54mm:PinHeader_1x03_P2.54mm_Vertical, symbol Device:Jumper_NC_Dual
- added R28, R29: 1k, Resistor_SMD:R_0603_1608Metric, symbol Device:R
- added unit 2 of SW1
- added SW3: SW_DP3T, RobotClub_footprint:CL-SB-13A-01, symbol Switch:SW_DP3T
- added SW4: SW_Push, Button_Switch_THT:SW_PUSH_6mm_H4.3mm, symbol Switch:SW_Push
- added SW5: SW_Coded_SH-7050, Button_Switch_THT:Nidec_Copal_SH-7010C, symbol Switch:SW_Coded_SH-7050
- added U10, U11, U15: 4_array, Resistor_SMD:R_Array_Convex_4x0603, symbol Resistance_array:4_array
- added U19: AP7361C-12E, Package_TO_SOT_SMD:TO-252-2, symbol Regulator_Linear:AP7361C-12E
- C10, C11: footprint (none) -> Capacitor_SMD:C_1210_3225Metric
- C12, C13, C14, C15, C6, C7, C8, C9: footprint (none) -> Capacitor_SMD:C_0603_1608Metric
- C4: value 220u -> 47u; footprint (none) -> Capacitor_SMD:C_Elec_6.3x5.4
- D1, D2, D3, D4, D5, D6: footprint (none) -> Diode_SMD:D_SOD-123
- D10, D7, D8, D9: footprint (none) -> Diode_SMD:D_SMA
- J1, J2: footprint (none) -> Connector_JST:JST_XH_S4B-XH-A-1_1x04_P2.50mm_Horizontal
- J3: renamed from J?; footprint (none) -> Connector_USB:USB_Mini_B_holes
- Q1, Q2, Q3, Q4: footprint (none) -> Package_TO_SOT_SMD:SOT-23
- R16, R17, R18, R19, R20, R21, R22, R23, R24, R25, R26, R27: footprint (none) -> Resistor_SMD:R_0603_1608Metric
- SW1: footprint (none) -> RobotClub_footprint:CL-SB-13A-01
- U7, U8: footprint (none) -> Display_7Segment:OSL10321
- Y1: footprint (none) -> Crystal:Crystal_SMD_SeikoEpson_FA238-4Pin_3.2x2.5mm
- gave numbers to parts that had none: 11
Connections:
- net input1 is gone; now on net Motor-PWM_1: R16.2, R18.2
- net input2 is gone; now on net Motor-PWM_2: R17.2, R19.2
- net +12V: now also C27.1, U19.3 (VO)
- net +24V: now also C22.1, C23.1, C24.1, C25.1, C26.1, F2.1, F3.1, U19.1 (VI)
- net +5V: now also C4.1, C5.1, U9.18 (AVCC), U9.4 (VCC), U9.6 (VCC), C19.2, C20.2, C21.1, D18.1 (VDD), F1.2, R28.1, R29.1, U10.1, U10.2, U10.3, U10.4, U11.1, U11.2, U11.3, U11.4; no longer J3.1 (VBUS)
- net GND: now also U17.3 (C), U18.3 (C), C19.1, C20.1, C21.2, D11.1 (K), D18.3 (VSS), D19.1 (K), D20.1 (K), H3.1, H4.1, SW4.1, SW5.C
- net GNDA: now also C22.2, C23.2, C24.2, C25.2, C26.2, C27.2, H1.1, H2.1, U19.2 (GND)
- net HL1: now also U9.28 (PC5(ADC5/SCL)(A5)), SW3.1
- net HL2: now also U9.27 (PC4(ADC4/SDA)(A4)), SW3.4
- net Input_Mode_Detect: now also J7.1 (Pin_1)
- net Latch_7seg_Driver: now also J6.1 (Pin_1)
- net Master_In_Slave_Out: now also J10.1 (Pin_1)
- net Master_Out_Slave_in: now also J11.1 (Pin_1)
- net Motor-PWM_1: now also J13.1 (Pin_1)
- net Motor-PWM_2: now also J12.1 (Pin_1)
- net Neo_Pixel: now also D18.4 (DIN), J14.1 (Pin_1)
- net Reset: now also R28.2, SW4.2
- net SW_1(Pull_Down_&_LED): now also D12.1 (K), SW5.1, U10.6
- net SW_2(Pull_Down_&_LED): now also D13.1 (K), SW5.2, U10.8
- net SW_3(Pull_Down_&_LED): now also D14.1 (K), SW5.4, U10.5
- net SW_4(Pull_Down_&_LED): now also D15.1 (K), SW5.8, U10.7
- net Serial_Clock: now also J9.1 (Pin_1)
- net Serial_Rx: now also J5.1 (Pin_1)
- net Slave_Select: now also J8.1 (Pin_1)
- net Software_Reset: now also J4.1 (Pin_1)
- net USB_Serial_D+: now also U15.8; no longer U14.5 (URx)
- net USB_Serial_D-: now also JP1.1, U15.7; no longer U14.6 (UTx), U9.30 (PD0(RXD)(D0/RX))
- net at U1.1 (QB): now also U3.3; no longer U3.2
- net at U1.15 (QA): now also U3.4; no longer U3.1
- net at U1.2 (QC): now also U3.2; no longer U3.3
- net at U1.3 (QD): now also U3.1; no longer U3.4
- net at U1.4 (QE): now also U4.4; no longer U4.1
- net at U1.5 (QF): now also U4.3; no longer U4.2
- net at U1.6 (QG): now also U4.2; no longer U4.3
- net at U1.7 (QH): now also U4.1; no longer U4.4
- net at R16.1: now also D19.2 (A); no longer U17.3 (C)
- net at R17.1: now also D20.2 (A); no longer U18.3 (C)
- net at U2.1 (QB): now also U5.3; no longer U5.2
- net at U2.15 (QA): now also U5.4; no longer U5.1
- net at U2.2 (QC): now also U5.2; no longer U5.3
- net at U2.3 (QD): now also U5.1; no longer U5.4
- net at U2.4 (QE): now also U6.4; no longer U6.1
- net at U2.5 (QF): now also U6.3; no longer U6.2
- net at U2.6 (QG): now also U6.2; no longer U6.3
- net at U2.7 (QH): now also U6.1; no longer U6.4
- net at SW2.2: now also SW3.3
- net at U3.8: now also U7.5 (D); no longer U7.1 (A)
- net at U3.7: now also U7.8 (C); no longer U7.10 (B)
- net at U3.6: now also U7.10 (B); no longer U7.8 (C)
- net at U3.5: now also U7.1 (A); no longer U7.5 (D)
- net at U4.8: now also U7.7 (DP8); no longer U7.4 (E)
- net at U4.7: now also U7.3 (G); no longer U7.2 (F)
- net at U4.6: now also U7.2 (F); no longer U7.3 (G)
- net at U4.5: now also U7.4 (E); no longer U7.7 (DP8)
- net at U5.8: now also U8.5 (D); no longer U8.1 (A)
- net at U5.7: now also U8.8 (C); no longer U8.10 (B)
- net at U5.6: now also U8.10 (B); no longer U8.8 (C)
- net at U5.5: now also U8.1 (A); no longer U8.5 (D)
- net at U6.8: now also U8.7 (DP8); no longer U8.4 (E)
- net at U6.7: now also U8.3 (G); no longer U8.2 (F)
- net at U6.6: now also U8.2 (F); no longer U8.3 (G)
- net at U6.5: now also U8.4 (E); no longer U8.7 (DP8)
- net at U14.2 (GP0): now also U16.3; no longer U16.1
- net at U14.3 (GP1): now also U16.4; no longer U16.2
- net at U14.7 (GP2): no longer U16.3
- net at U14.8 (GP3): no longer U16.4
- net at U16.8: no longer D16.2 (A)
- net at U16.7: no longer D17.2 (A)
- net at U16.6: now also D16.2 (A)
- net at U16.5: now also D17.2 (A)
- new net: F1.1, J3.1 (VBUS)
- new net: U14.5 (URx), U15.1
- new net: U14.6 (UTx), U15.2
- new net: D11.2 (A), R29.2
- new net: D12.2 (A), U11.8
- new net: D13.2 (A), U11.7
- new net: D14.2 (A), U11.6
- new net: D15.2 (A), U11.5
- new net +BATT: F2.2, F3.2
- new net USB_Serial_D-(lock): JP1.2, U9.30 (PD0(RXD)(D0/RX))
- no-connect marks 8 -> 23
Other:
- note removed: "DIP*4\n"
- note removed: "slide*2\n"
- moved on the sheet: C1, C10, C11, C12, C13, C14, C15, C16, C17, C18, C2, C3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
